File: schematics/openegg2.sch (EAGLE design)
At the start: 69 parts, among them IC1 L5973D, IC2 ZLDO330, J1 22-27-2031-03, Q1 BC846, Q2 BC846, Q3 BC846, Q4 BC846, Q6 BC856, Q8 BC846, X2 32.768KHz

Commit message: Undo wrong checkin
Parts:
- removed L4: 1uH, rcl:L-EUL1812
- added C15: 100uF, rcl:CPOL-US153CLV-0505
- added F2: 3A, rcl:R-EU_R2010
- added VR2: 4.5V, varistor:VARISTORCN1812
- C2: value 100uF -> 10uF ceramic; device rcl:CPOL-EU140CLH-1014 -> rcl:C-EUC1210K
- C9: value 30uF -> 470uF; device rcl:CPOL-EU140CLH-1014 -> rcl:CPOL-USCT7343
- VR1: device varistor:VARISTORCN1206 -> rcl:R-EU_R2010
Connections:
- net +12V: now also C15.+, C2.1; no longer C2.+
- net GND: now also C15.-, C2.2, VR2.1; no longer C2.-
- net N$13: now also F2.1; no longer L4.2
- net V+: now also F2.2, VR2.2; no longer L4.1
Other:
- moved on the sheet: C9
Changed lines of the file:
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@@
 <part name="IC1" library="st-microelectronics" deviceset="L5973D" device=""/>
 <part name="L2" library="inductors-2" deviceset="DR127" device="" value="15uH"/>
-<part name="L4" library="rcl" deviceset="L-EU" device="L1812" value="1uH"/>
 <part name="P+3" library="supply1" deviceset="+12V" device=""/>
-<part name="C2" library="rcl" deviceset="CPOL-EU" device="140CLH-1014" value="100uF"/>
-<part name="C9" library="rcl" deviceset="CPOL-EU" device="140CLH-1014" value="30uF"/>
 <part name="GND9" library="supply1" deviceset="GND" device=""/>
 <part name="GND11" library="supply1" deviceset="GND" device=""/>
@@
 <part name="GND37" library="supply1" deviceset="GND" device=""/>
 <part name="P+5" library="supply1" deviceset="V+" device="" value="+3.6V"/>
-<part name="VR1" library="varistor" deviceset="VARISTOR" device="CN1206" value="18V"/>
+<part name="VR1" library="rcl" deviceset="R-EU_" device="R2010" value="18V"/>
 <part name="GND38" library="supply1" deviceset="GND" device=""/>
 <part name="GND39" library="supply1" deviceset="GND" device=""/>
@@
 <part name="R7" library="rcl" deviceset="R-EU_" device="R0603" value="10k"/>
 <part name="R25" library="rcl" deviceset="R-EU_" device="R0603" value="10k"/>
+<part name="C2" library="rcl" deviceset="C-EU" device="C1210K" value="10uF ceramic"/>
+<part name="C9" library="rcl" deviceset="CPOL-US" device="CT7343" value="470uF"/>
+<part name="C15" library="rcl" deviceset="CPOL-US" device="153CLV-0505" value="100uF"/>
+<part name="GND10" library="supply1" deviceset="GND" device=""/>
+<part name="VR2" library="varistor" deviceset="VARISTOR" device="CN1812" value="4.5V"/>
+<part name="F2" library="rcl" deviceset="R-EU_" device="R2010" value="3A"/>
+<part name="GND15" library="supply1" deviceset="GND" device=""/>
 </parts>
 <sheets>
@@
 <instance part="IC1" gate="G$1" x="312.42" y="132.08"/>
 <instance part="L2" gate="G$1" x="337.82" y="139.7" rot="R270"/>
-<instance part="L4" gate="G$1" x="345.44" y="137.16"/>
 <instance part="P+3" gate="1" x="287.02" y="144.78"/>
-<instance part="C2" gate="G$1" x="292.1" y="149.86" rot="R180"/>
-<instance part="C9" gate="G$1" x="340.36" y="124.46"/>
 <instance part="GND9" gate="1" x="292.1" y="162.56" rot="R180"/>
 <instance part="GND11" gate="1" x="330.2" y="132.08"/>
-<instance part="GND12" gate="1" x="340.36" y="116.84"/>
+<instance part="GND12" gate="1" x="340.36" y="109.22"/>
 <instance part="GND13" gate="1" x="327.66" y="116.84"/>
 <instance part="C11" gate="G$1" x="284.48" y="134.62" rot="R270"/>
@@
 <instance part="+3V9" gate="G$1" x="109.22" y="104.14" rot="R90"/>
 <instance part="+3V10" gate="G$1" x="200.66" y="104.14" rot="R270"/>
-<instance part="P+6" gate="1" x="345.44" y="147.32"/>
+<instance part="P+6" gate="1" x="350.52" y="152.4"/>
 <instance part="+3V12" gate="G$1" x="322.58" y="93.98"/>
 <instance part="IC1" gate="-EXP" x="312.42" y="154.94"/>
@@
 <instance part="GND37" gate="1" x="134.62" y="172.72"/>
 <instance part="P+5" gate="1" x="134.62" y="213.36"/>
-<instance part="VR1" gate="G$1" x="226.06" y="17.78" rot="R90"/>
+<instance part="VR1" gate="G$1" x="226.06" y="17.78" rot="R270"/>
 <instance part="GND38" gate="1" x="226.06" y="7.62"/>
 <instance part="GND39" gate="1" x="208.28" y="142.24" rot="R90"/>
@@
 <instance part="R7" gate="G$1" x="124.46" y="7.62" rot="R180"/>
 <instance part="R25" gate="G$1" x="124.46" y="0" rot="R180"/>
+<instance part="C2" gate="G$1" x="292.1" y="149.86" rot="R180"/>
+<instance part="C9" gate="G$1" x="340.36" y="121.92"/>
+<instance part="C15" gate="G$1" x="297.18" y="149.86" rot="R180"/>
+<instance part="GND10" gate="1" x="297.18" y="162.56" rot="R180"/>
+<instance part="VR2" gate="G$1" x="358.14" y="121.92" rot="R270"/>
+<instance part="F2" gate="G$1" x="350.52" y="139.7" rot="R90"/>
+<instance part="GND15" gate="1" x="358.14" y="109.22"/>
 </instances>
 <busses>
@@
 </segment>
 <segment>
-<pinref part="C2" gate="G$1" pin="-"/>
 <pinref part="GND9" gate="1" pin="GND"/>
 <wire x1="292.1" y1="154.94" x2="292.1" y2="160.02" width="0.1524" layer="91"/>
-</segment>
-<segment>
-<pinref part="C9" gate="G$1" pin="-"/>
-<pinref part="GND12" gate="1" pin="GND"/>
+<pinref part="C2" gate="G$1" pin="2"/>
 </segment>
 <segment>
@@
 <pinref part="GND8" gate="1" pin="GND"/>
 <wire x1="350.52" y1="55.88" x2="350.52" y2="60.96" width="0.1524" layer="91"/>
+</segment>
+<segment>
+<pinref part="C15" gate="G$1" pin="-"/>
+<pinref part="GND10" gate="1" pin="GND"/>
+<wire x1="297.18" y1="160.02" x2="297.18" y2="154.94" width="0.1524" layer="91"/>
+</segment>
+<segment>
+<pinref part="GND12" gate="1" pin="GND"/>
+<pinref part="C9" gate="G$1" pin="-"/>
+<wire x1="340.36" y1="111.76" x2="340.36" y2="116.84" width="0.1524" layer="91"/>
+</segment>
+<segment>
+<pinref part="VR2" gate="G$1" pin="1"/>
+<pinref part="GND15" gate="1" pin="GND"/>
+<wire x1="358.14" y1="111.76" x2="358.14" y2="116.84" width="0.1524" layer="91"/>
 </segment>
 </net>
@@
 </segment>
 <segment>
-<pinref part="L4" gate="G$1" pin="1"/>
-<pinref part="P+6" gate="1" pin="V+"/>
-<wire x1="345.44" y1="144.78" x2="345.44" y2="142.24" width="0.1524" layer="91"/>
-</segment>
-<segment>
 <pinref part="R24" gate="G$1" pin="1"/>
 <pinref part="P+5" gate="1" pin="V+"/>
 <wire x1="134.62" y1="210.82" x2="134.62" y2="208.28" width="0.1524" layer="91"/>
 </segment>
+<segment>
+<pinref part="F2" gate="G$1" pin="2"/>
+<pinref part="P+6" gate="1" pin="V+"/>
+<wire x1="350.52" y1="149.86" x2="350.52" y2="147.32" width="0.1524" layer="91"/>
+<pinref part="VR2" gate="G$1" pin="2"/>
+<wire x1="350.52" y1="147.32" x2="350.52" y2="144.78" width="0.1524" layer="91"/>
+<wire x1="358.14" y1="127" x2="358.14" y2="144.78" width="0.1524" layer="91"/>
+<wire x1="358.14" y1="144.78" x2="358.14" y2="147.32" width="0.1524" layer="91"/>
+<wire x1="358.14" y1="147.32" x2="350.52" y2="147.32" width="0.1524" layer="91"/>
+<junction x="350.52" y="147.32"/>
+</segment>
 </net>
 <net name="N$13" class="0">
 <segment>
-<pinref part="L4" gate="G$1" pin="2"/>
-<wire x1="345.44" y1="132.08" x2="345.44" y2="129.54" width="0.1524" layer="91"/>
 <pinref part="L2" gate="G$1" pin="2"/>
-<wire x1="345.44" y1="129.54" x2="340.36" y2="129.54" width="0.1524" layer="91"/>
+<wire x1="350.52" y1="129.54" x2="340.36" y2="129.54" width="0.1524" layer="91"/>
 <wire x1="340.36" y1="129.54" x2="337.82" y2="129.54" width="0.1524" layer="91"/>
 <wire x1="337.82" y1="129.54" x2="337.82" y2="132.08" width="0.1524" layer="91"/>
-<pinref part="C9" gate="G$1" pin="+"/>
-<wire x1="340.36" y1="127" x2="340.36" y2="129.54" width="0.1524" layer="91"/>
+<wire x1="340.36" y1="124.46" x2="340.36" y2="129.54" width="0.1524" layer="91"/>
 <junction x="340.36" y="129.54"/>
 <pinref part="R9" gate="G$1" pin="1"/>
@@
 <wire x1="335.28" y1="129.54" x2="337.82" y2="129.54" width="0.1524" layer="91"/>
 <junction x="337.82" y="129.54"/>
+<pinref part="C9" gate="G$1" pin="+"/>
+<pinref part="F2" gate="G$1" pin="1"/>
+<wire x1="350.52" y1="134.62" x2="350.52" y2="129.54" width="0.1524" layer="91"/>
 </segment>
 </net>
@@
 <pinref part="P+3" gate="1" pin="+12V"/>
 <pinref part="IC1" gate="G$1" pin="VCC"/>
-<wire x1="299.72" y1="142.24" x2="292.1" y2="142.24" width="0.1524" layer="91"/>
-<pinref part="C2" gate="G$1" pin="+"/>
+<wire x1="299.72" y1="142.24" x2="297.18" y2="142.24" width="0.1524" layer="91"/>
+<wire x1="297.18" y1="142.24" x2="292.1" y2="142.24" width="0.1524" layer="91"/>
 <wire x1="292.1" y1="147.32" x2="292.1" y2="142.24" width="0.1524" layer="91"/>
 <junction x="292.1" y="142.24"/>
 <wire x1="292.1" y1="142.24" x2="287.02" y2="142.24" width="0.1524" layer="91"/>
-</segment>
-<segment>
+<pinref part="C2" gate="G$1" pin="1"/>
+<pinref part="C15" gate="G$1" pin="+"/>
+<wire x1="297.18" y1="147.32" x2="297.18" y2="142.24" width="0.1524" layer="91"/>
+<junction x="297.18" y="142.24"/>
+</segment>
+<segment>

Commit message: Route button pull up resistors.
Parts:
- removed R25, R5, R6, R7: 10k, rcl:R-EU_R0603
- added RN1: (no value), resistor-array:742-8_S
Connections:
- net +3V3: now also RN1A.2, RN1B.2, RN1C.2, RN1D.2; no longer R25.2, R5.2, R6.2, R7.2
- net B0: now also RN1B.1; no longer R25.1
- net B1: now also RN1A.1; no longer R7.1
- net B2: now also RN1D.1; no longer R6.1
- net B3: now also RN1C.1; no longer R5.1
Changed lines of the file:
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@@
 <layer number="53" name="tGND_GNDA" color="7" fill="9" visible="no" active="no"/>
 <layer number="54" name="bGND_GNDA" color="1" fill="9" visible="no" active="no"/>
+<layer number="56" name="wert" color="7" fill="1" visible="no" active="no"/>
 <layer number="91" name="Nets" color="2" fill="1" visible="yes" active="yes"/>
 <layer number="92" name="Busses" color="1" fill="1" visible="yes" active="yes"/>
@@
 <layer number="131" name="tAdjust" color="7" fill="1" visible="no" active="yes"/>
 <layer number="132" name="bAdjust" color="7" fill="1" visible="no" active="yes"/>
+<layer number="150" name="Notes" color="7" fill="1" visible="yes" active="yes"/>
+<layer number="151" name="HeatSink" color="14" fill="1" visible="no" active="no"/>
 <layer number="200" name="200bmp" color="7" fill="1" visible="no" active="yes"/>
 <layer number="201" name="201bmp" color="7" fill="1" visible="no" active="yes"/>
@@
 <part name="GND8" library="supply1" deviceset="GND" device=""/>
 <part name="+3V13" library="supply1" deviceset="+3V3" device=""/>
-<part name="R5" library="rcl" deviceset="R-EU_" device="R0603" value="10k"/>
-<part name="R6" library="rcl" deviceset="R-EU_" device="R0603" value="10k"/>
-<part name="R7" library="rcl" deviceset="R-EU_" device="R0603" value="10k"/>
-<part name="R25" library="rcl" deviceset="R-EU_" device="R0603" value="10k"/>
 <part name="C2" library="rcl" deviceset="C-EU" device="C1210K" value="10uF ceramic"/>
 <part name="C9" library="rcl" deviceset="CPOL-US" device="CT7343" value="470uF"/>
@@
 <part name="F2" library="rcl" deviceset="R-EU_" device="R2010" value="3A"/>
 <part name="GND15" library="supply1" deviceset="GND" device=""/>
+<part name="RN1" library="resistor-array" deviceset="742-8_S" device=""/>
 </parts>
 <sheets>
@@
 <instance part="GND8" gate="1" x="350.52" y="53.34"/>
 <instance part="+3V13" gate="G$1" x="116.84" y="30.48"/>
-<instance part="R5" gate="G$1" x="124.46" y="22.86" rot="R180"/>
-<instance part="R6" gate="G$1" x="124.46" y="15.24" rot="R180"/>
-<instance part="R7" gate="G$1" x="124.46" y="7.62" rot="R180"/>
-<instance part="R25" gate="G$1" x="124.46" y="0" rot="R180"/>
 <instance part="C2" gate="G$1" x="292.1" y="149.86" rot="R180"/>
 <instance part="C9" gate="G$1" x="340.36" y="121.92"/>
@@
 <instance part="F2" gate="G$1" x="350.52" y="139.7" rot="R90"/>
 <instance part="GND15" gate="1" x="358.14" y="109.22"/>
+<instance part="RN1" gate="A" x="124.46" y="7.62" rot="R180"/>
+<instance part="RN1" gate="B" x="124.46" y="0" rot="R180"/>
+<instance part="RN1" gate="C" x="124.46" y="22.86" rot="R180"/>
+<instance part="RN1" gate="D" x="124.46" y="15.24" rot="R180"/>
 </instances>
 <busses>
@@
 </segment>
 <segment>
-<pinref part="R25" gate="G$1" pin="2"/>
 <wire x1="119.38" y1="0" x2="116.84" y2="0" width="0.1524" layer="91"/>
 <wire x1="116.84" y1="0" x2="116.84" y2="7.62" width="0.1524" layer="91"/>
-<pinref part="R7" gate="G$1" pin="2"/>
 <wire x1="116.84" y1="7.62" x2="119.38" y2="7.62" width="0.1524" layer="91"/>
-<pinref part="R6" gate="G$1" pin="2"/>
 <wire x1="119.38" y1="15.24" x2="116.84" y2="15.24" width="0.1524" layer="91"/>
 <wire x1="116.84" y1="15.24" x2="116.84" y2="7.62" width="0.1524" layer="91"/>
 <junction x="116.84" y="7.62"/>
-<pinref part="R5" gate="G$1" pin="2"/>
 <wire x1="119.38" y1="22.86" x2="116.84" y2="22.86" width="0.1524" layer="91"/>
 <wire x1="116.84" y1="22.86" x2="116.84" y2="15.24" width="0.1524" layer="91"/>
@@
 <wire x1="116.84" y1="22.86" x2="116.84" y2="27.94" width="0.1524" layer="91"/>
 <junction x="116.84" y="22.86"/>
+<pinref part="RN1" gate="A" pin="2"/>
+<pinref part="RN1" gate="B" pin="2"/>
+<pinref part="RN1" gate="C" pin="2"/>
+<pinref part="RN1" gate="D" pin="2"/>
 </segment>
 </net>
@@
 <pinref part="B0" gate="G$1" pin="P"/>
 <wire x1="154.94" y1="22.86" x2="154.94" y2="20.32" width="0.1524" layer="91"/>
-<pinref part="R25" gate="G$1" pin="1"/>
 <wire x1="154.94" y1="20.32" x2="154.94" y2="17.78" width="0.1524" layer="91"/>
 <wire x1="129.54" y1="0" x2="147.32" y2="0" width="0.1524" layer="91"/>
@@
 <wire x1="147.32" y1="20.32" x2="154.94" y2="20.32" width="0.1524" layer="91"/>
 <junction x="154.94" y="20.32"/>
+<pinref part="RN1" gate="B" pin="1"/>
 </segment>
 <segment>
@@
 <pinref part="B1" gate="G$1" pin="P"/>
 <wire x1="172.72" y1="22.86" x2="172.72" y2="20.32" width="0.1524" layer="91"/>
-<pinref part="R7" gate="G$1" pin="1"/>
 <wire x1="172.72" y1="20.32" x2="172.72" y2="17.78" width="0.1524" layer="91"/>
 <wire x1="129.54" y1="7.62" x2="167.64" y2="7.62" width="0.1524" layer="91"/>
@@
 <wire x1="167.64" y1="20.32" x2="172.72" y2="20.32" width="0.1524" layer="91"/>
 <junction x="172.72" y="20.32"/>
+<pinref part="RN1" gate="A" pin="1"/>
 </segment>
 <segment>
@@
 <pinref part="B2" gate="G$1" pin="P"/>
 <wire x1="187.96" y1="22.86" x2="187.96" y2="20.32" width="0.1524" layer="91"/>
-<pinref part="R6" gate="G$1" pin="1"/>
 <wire x1="187.96" y1="20.32" x2="187.96" y2="17.78" width="0.1524" layer="91"/>
 <wire x1="129.54" y1="15.24" x2="185.42" y2="15.24" width="0.1524" layer="91"/>
@@
 <wire x1="185.42" y1="20.32" x2="187.96" y2="20.32" width="0.1524" layer="91"/>
 <junction x="187.96" y="20.32"/>
+<pinref part="RN1" gate="D" pin="1"/>
 </segment>
 <segment>
@@
 <pinref part="B3" gate="G$1" pin="P"/>
 <wire x1="203.2" y1="22.86" x2="203.2" y2="20.32" width="0.1524" layer="91"/>
-<pinref part="R5" gate="G$1" pin="1"/>
 <wire x1="203.2" y1="20.32" x2="203.2" y2="17.78" width="0.1524" layer="91"/>
 <wire x1="129.54" y1="22.86" x2="147.32" y2="22.86" width="0.1524" layer="91"/>
@@
 <wire x1="198.12" y1="20.32" x2="203.2" y2="20.32" width="0.1524" layer="91"/>
 <junction x="203.2" y="20.32"/>
-</segment>
-<segment>
+<pinref part="RN1" gate="C" pin="1"/>
+</segment>
+<segment>
